File: Hardware/Processor_Periph/Processor.sch (KiCad schematic (older format))
At the start: 96 parts, among them J1 5V, J2 UART0, J3 USB_OTG, J4 JTAGICE3-SWD, Q1 BSSB06NE, Q2 BSSB06NE, Q3 BSSB06NE, Q4 BSSB06NE, SW1 PB, SW2 PB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

Commit message: Added SRAM and microSD card to design
Parts:
- added J?: Micro_SD_Card, symbol Micro_SD_Card
- added Q?: BSSB06NE, TO_SOT_Packages_SMD:SOT-23, symbol Q_NMOS_GSD
- added R?: 27R, Capacitors_SMD:C_0603, symbol R
- added R?: 10k, Capacitors_SMD:C_0603, symbol R
- added U?: CY7C1018, symbol CY7C1018
Connections:
- net labels added: EBI
- net labels removed: RAM_ADDR, RAM_DATA
- wire segments 508 -> 407
Other:
- note removed: "SD Card Interface"
- moved on the sheet: C10, C11, C15, C19, C20, C4, C5, C9, J1, J2, J3, JP1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

Commit message: Added & Routed RAM. Made changes to documentation file structure. Added more datasheets
Parts:
- removed R11: 27R, Capacitors_SMD:C_0603, symbol R
- removed U2: ATSAM4E16E, Housings_QFP:TQFP-144_20x20mm_Pitch0.5mm, symbol ATSAM4E16E-RESCUE-Processor
- added C? (x3): 100nF, Capacitors_SMD:C_0603, symbol C
- added C?: 4.7uF, Capacitors_SMD:C_0805, symbol C
- added R? (x4): 10k, Capacitors_SMD:C_0603, symbol R
- added U?: ATSAM4E16E, symbol ATSAM4E16E
- Q1, Q2, Q3, Q4, Q?: value BSSB06NE -> BSS806NE
Connections:
- net labels added: SD_EN
- net labels removed: ~WAIT
- wire segments 407 -> 641
Other:
- moved on the sheet: C1, C10, C11, C12, C13, C14, C15, C16, C17, C18, C19, C2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

Commit message: Added flash, minor schematic tweaks, regenerated PDFs, added more ref stuff, updated todo
Parts:
- removed R?: 10k, Capacitors_SMD:C_0603, symbol R
- added C?: 4.5nF, Capacitors_SMD:C_0603, symbol C
- added C? (x2): 100nF, Capacitors_SMD:C_0603, symbol C
- added J?: PWM, symbol CONN_02X04
- added R?: 27R, Capacitors_SMD:C_0603, symbol R
- added U?: S25FL127S, symbol S25FL127S
Connections:
- net labels added: MCCK_R, MII, NVM_MISO, NVM_MOSI, NVM_SCK, NVM_SCK_R, NVM_~CS, NVM_~HOLD, PWM, RAM_~CS, RAM_~RD, RAM_~WE, USBD_R+, USBD_R-
- net labels removed: DD+, DD-, ~CS0, ~RD, ~WE
- wire segments 641 -> 729
- no-connect marks 5 -> 6
Other:
- note added: "Remove local KiCad Libs from past projects.\nNeed to add:\nEthernet PHY, Magnetics, & RJ45\nBreakout Connectors\n"
- note added: "TODO: ADD ETHERNET PHY (MII INTERFACE)"
- note added: "TODO: ADD PULLUPS ON THESE SIGNALS"
- note added: "TODO: CHECK !WP AND OTHER DISCRETES HERE"
- note removed: "Ethernet MII interface"
- note removed: "Remove local KiCad Libs from past projects.\nNeed to add:\nEEPROM\nRAM\nEthernet PHY, Magnetics, & RJ45\nSD Card\nBreakout Connectors\n"
- note removed: "Stepper Motor Control"
- moved on the sheet: C1, C10, C11, C12, C13, C14, C15, C16, C17, C18, C19, C2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
