File: Hardware/Processor_Periph/Processor.sch (KiCad schematic (older format))
At the start: 115 parts, among them J1 5V, J2 UART0, J3 USB_OTG, J4 JTAGICE3-SWD, Q1 BSS806NE, Q2 BSS806NE, Q3 BSS806NE, Q4 BSS806NE, SW1 PB, SW2 PB, SW3 ~RST, U1 TXS0102, U3 3.0V, U4 LM3671, U5 PRTR5V0U2X, Y1 32.768kHz, Y2 12MHz

Commit message: Added design_notes and preliminary KiCad style guide
Parts:
- added C? (x2): ?pF, Capacitors_SMD:C_0603, symbol C
- added C?: 10uF, Capacitors_SMD:C_0805, symbol C
- added C? (x3): 100nF, Capacitors_SMD:C_0603, symbol C
- added J?: RJ45-TRANSFO, symbol RJ45-TRANSFO
- added R? (x3): 0R, Capacitors_SMD:C_0603, symbol R
- added R?: 4.87k, symbol R
- added Y?: 25MHz, Crystals:Crystal_HC49-SD_SMD, symbol Crystal
Connections:
- net GND: now also C?.2, C?.2, C?.2, C?.2, C?.2, C?.2
- net PCLK: now reaches U?.144 (PB13/PWML2/PCK0/SCK0/DAC0)
- net ERX-: now reaches U?.13 (RD-)
- net ERX-: now also U?.14 (RD+), J?.4 (RD+), J?.6 (RD-)
- net ETX-: now reaches U?.16 (TD-)
- net ETX-: now also J?.3 (TD-)
- net ETX+: now reaches U?.17 (TD+)
- net ETX+: now also J?.1 (TD+)
- net at U?.18 (PFBIN1): now also C?.1
- net at U?.23 (PFBOUT): now also C?.1, C?.1
- net at U?.33 (X2): now also R?.2
- net at U?.34 (X1): now also R?.2, R?.2
- net at U?.37 (PFBIN2): now also C?.1
- new net: C?.1, R?.1, Y?.1
- new net: C?.1, R?.1, Y?.2
- new net CLK_25: R?.1
Other:
- note added: "DNP"
- note added: "TODO: CHECK THESE CAPACITOR VALUES, THEY SEEM A BIT HIGH."
- moved on the sheet: U?

Commit message: Added more detail to style guide. Generated in progress schematic PDF
Connections:
- net NVM_SCK: now also R?.2, U?.6 (CLK); no longer R?.1, U?.51 (PA14/SPCK/PWMH3/WKUP8)
- net NVM_SCK_R: now also R?.1, U?.51 (PA14/SPCK/PWMH3/WKUP8); no longer R?.2, U?.6 (CLK)

Commit message: Added design notes, cleaned up sch
Parts:
- removed C? (x2): ?pF, Capacitors_SMD:C_0603, symbol C
- removed R? (x3): 0R, Capacitors_SMD:C_0603, symbol R
- removed R?: 4.87k, symbol R
- removed Y?: 25MHz, Crystals:Crystal_HC49-SD_SMD, symbol Crystal
- added C? (x4): 100nF, Capacitors_SMD:C_0603, symbol C
- added C?: 1.5nF, Capacitors_SMD:C_0603, symbol C
- added R? (x4): 49.9R, symbol R
Connections:
- net +3V3: now also J?.2 (TCT), J?.5 (RCT), C?.1, C?.1, C?.1, R?.1, R?.1, R?.2, R?.2
- net ERX-: now also R?.1, R?.1
- net ETX+: now also R?.2
- net ETX-: now also R?.2
- net GND: now also C?.2, C?.2, C?.2, C?.2
- net at J?.8: now also C?.1
- no-connect marks 6 -> 7
Other:
- note removed: "DNP"
- moved on the sheet: C?, J?, U?

Commit message: Finished Schematic Draft
Parts:
- removed C19, C20: 12pF, Capacitors_SMD:C_0603, symbol C
- removed C?: 4.5nF, Capacitors_SMD:C_0603, symbol C
- removed C?: 100nF, Capacitors_SMD:C_0603, symbol C
- removed C?: 1.5nF, Capacitors_SMD:C_0603, symbol C
- removed J?: RJ45-TRANSFO, symbol RJ45-TRANSFO
- removed Q?: BSS806NE, TO_SOT_Packages_SMD:SOT-23, symbol Q_NMOS_GSD
- removed R?: 10k, Capacitors_SMD:C_0603, symbol R
- removed Y2: 12MHz, Crystals:Crystal_HC49-SD_SMD, symbol Crystal
- added C? (x4): 100nF, Capacitors_SMD:C_0603, symbol C
- added C? (x2): 1uF, Capacitors_SMD:C_0603, symbol C
- added C?: 10uF, Capacitors_SMD:C_0603, symbol C
- added C? (x2): 10nF, Capacitors_SMD:C_0603, symbol C
- added J?: RJ-45_J0006D01BNL, symbol RJ-45_J0006D01BNL
- added J?: I2C, symbol CONN_01X03
- added R? (x13): 10k, Capacitors_SMD:C_0603, symbol R
- added R? (x2): 120R, Capacitors_SMD:C_0603, symbol R
- added R?: 1.5K, Capacitors_SMD:C_0603, symbol R
- added R?: 4.87k, symbol R
- added R? (x26): 2.2k, Capacitors_SMD:C_0603, symbol R
- added TP?: 1V8, Measurement_Points:Measurement_Point_Round-SMD-Pad_Small, symbol TEST
- added TP?: LED_SPEED, Measurement_Points:Measurement_Point_Round-SMD-Pad_Small, symbol TEST
- added U?: DSC61XX, symbol DSC61XX
- added U?: MIC5365, symbol MIC5365
- added U?: Oscillator, symbol Oscillator
- R14, R17, R19, R21: value 150R -> 120R
Connections:
- net VBUS is gone; now on net +5V: C5.1, J3.1 (VBUS), JP1.3, R2.2, U5.4 (A)
- net +3V3: now also C?.1, R?.1, U?.22 (AVDD33), U?.32 (IOVDD33), U?.48 (IOVDD33), C?.1, C?.1, C?.1, C?.1, C?.1, C?.1, J?.4 (TCT), J?.5 (RCT), R?.1, R?.1, R?.1, R?.1, R?.1, R?.1, R?.1, R?.1, R?.1, R?.1, R?.1, R?.1, R?.1, R?.1, R?.1, R?.1, R?.1, R?.1, R?.1, R?.1, R?.1, R?.1, R?.1, R?.1, R?.1, R?.2, R?.2, U?.1 (VIN), U?.4 (VDD)
- net ERX-: now also J?.3 (RD+), J?.6 (RD-)
- net ETX+: now also J?.1 (TD+)
- net ETX-: now also J?.2 (TD-)
- net GCOL: now also R?.1, R?.2
- net GCRS: now also R?.1, R?.2
- net GMDIO: now also R?.2
- net GND: now also C?.2, J?.6 (VSS), U?.15 (AGND), U?.19 (AGND), U?.35 (IOGND), U?.36 (DGND), U?.47 (IOGND), C?.2, C?.2, C?.2, C?.2, C?.2, C?.2, C?.2, C?.2, C?.2, J?.1 (P1), J?.8, R?.1, R?.1, R?.2, R?.2, R?.2, R?.2, R?.2, R?.2, R?.2, R?.2, R?.2, R?.2, R?.2, R?.2, R?.2, U?.2 (GND), U?.2 (GND), U?.2 (GND); no longer R?.2
- net GRX0: now also R?.1, R?.2
- net GRX1: now also R?.1, R?.2
- net GRX2: now also R?.1, R?.2
- net GRX3: now also R?.1, R?.2
- net GRXDV: now also R?.1, R?.2
- net GRXER: now also R?.1, R?.2
- net GTX3: now also R?.1, R?.2
- net MCCDA2: now also R?.2
- net MCCDA3: now also R?.2
- net MCDA0: now also R?.2
- net MCDA1: now also R?.2
- net RAM_~WE: now also R?.2; no longer R?.1
- net XIN: now also U?.1 (OUT)
- net PHY_~INT: now reaches U?.67 (NCS3/PD19)
- net PHY_~INT: now also U?.7 (PWR_DOWN/INT), R?.2
- net PHY_~RST: now reaches U?.69 (NCS1/PD18)
- net PHY_~RST: now also U?.29 (~RESET~), R?.2
- net I2C_SCL: now reaches U?.77 (PA4/TWCK0/TCLK0/WKUP3)
- net I2C_SCL: now also J?.3 (P3), R?.2, R?.2
- net I2C_SDA: now reaches U?.91 (PA3/TWD0/NPCS3)
- net I2C_SDA: now also J?.2 (P2), R?.2, R?.2
- net PFBIN1: now reaches C?.1, U?.18 (PFBIN1)
- net at U?.20 (RESERVED): now also R?.1
- net at U?.21 (RESERVED): now also R?.1
- net PFBOUT: now reaches C?.1, C?.1, U?.23 (PFBOUT)
- net RBIAS: now reaches U?.24 (RBIAS)
- net RBIAS: now also R?.1
- net LED_ACT: now reaches U?.26 (AN_EN/LED_ACT/COL)
- net LED_ACT: now also J?.12 (LEDY_A), R?.1, R?.2
- net LED_SP: now reaches U?.27 (AN1/LED_SPEED)
- net LED_SP: now also R?.1, R?.2, TP?.1
- net LED_LN: now reaches U?.28 (AN0/LED_LINK)
- net LED_LN: now also J?.9 (LEDG_A), R?.1, R?.2
- net at U?.34 (X1): now also U?.3 (OUT)
- net PFBIN2: now reaches C?.1, U?.37 (PFBIN2)
- net GTXER: no longer names the net of U?.74 (GTXER/PD17)
- net SD_EN: no longer names the net of U?.59 (PA25/CTS1/PWMH2/A23/PIODC1)
- net XOUT: no longer names the net of U?.141 (PB8/XOUT)
- new net: R?.2, U?.1 (OUT)
- new net: J?.10 (LEDG_K), R?.2
- new net: J?.11 (LEDY_K), R?.2
- new net: R?.2, U?.1 (EN)
- new net +1V8: C?.1, C?.1, C?.1, R?.1, TP?.1, U?.5 (VOUT)
- new net LDO_EN: R?.2, U?.3 (EN)
- no-connect marks 7 -> 10
Other:
- note added: "AN_0"
- note added: "AN_1"
- note added: "AN_EN"
- note added: "LED_CFG"
- note added: "MDIX_EN"
- note added: "MII_MODE"
- note added: "PHY Strapping Options"
- note added: "PHY_ADDR[0]"
- note added: "PHY_ADDR[1]"
- note added: "PHY_ADDR[2]"
- note added: "PHY_ADDR[3]"
- note added: "PHY_ADDR[4]"
- note added: "SNI_MODE"
- note removed: "Remove local KiCad Libs from past projects.\nNeed to add:\nEthernet PHY, Magnetics, & RJ45\nBreakout Connectors\n"
- note removed: "TODO: ADD PULLUPS ON THESE SIGNALS"
- note removed: "TODO: CHECK !WP AND OTHER DISCRETES HERE"
- moved on the sheet: C38, C39, C?, D1, D2, D3, D4, Q1, Q2, Q3, Q4, R12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

Commit message: Added breakout connectors, ran ERC & corrected minor issues
Parts:
- added J?: Spare0, symbol CONN_02X08
- added J?: Spare1, symbol CONN_02X08
- C4: renamed from C10; value 27pF -> 3.9pF
- C5: renamed from C11; value 27pF -> 3.9pF
- gave numbers to parts that had none: 88
- renumbered C9 to C1, C1 to C13, C2 to C16, C3 to C17, C6 to C18, C7 to C19, C40 to C2, C8 to C20, C12 to C22, C13 to C23, C14 to C24, C16 to C26, C17 to C27, C18 to C28, C15 to C3, C21 to C31, C22 to C32, C23 to C33, C24 to C35, C25 to C36, C26 to C37, C27 to C39, C28 to C40, C30 to C47, C31 to C48, C32 to C49, C33 to C50, C34 to C51, C35 to C52, C36 to C53, C37 to C54, C38 to C57, C39 to C58, C4 to C6, C5 to C7, C41 to C9, D5 to D1, D1 to D2, D2 to D3, D3 to D4, D4 to D5, J2 to J1, J1 to J2, J4 to J8, L2 to L1, L1 to L2, R1 to R2, R6 to R29, R2 to R3, R7 to R30, R8 to R31, R9 to R32, R12 to R37, R10 to R39, R3 to R4, R15 to R41, R13 to R43, R14 to R48, R4 to R5, R16 to R53, R17 to R54, R18 to R59, R5 to R6, R19 to R64, R20 to R65, R22 to R7, R21 to R70, SW3 to SW1, SW1 to SW3, TP8 to TP10, TP3 to TP2, TP2 to TP4, TP4 to TP5, TP5 to TP6, TP6 to TP7, TP7 to TP8, U4 to U2, U5 to U4, U3 to U9
Connections:
- net labels added: MCU_XIN, PA0, PA1, PA16, PA17, PA2, PA21, PA22, PA23, PA24, PA25, PA5, PA6, PB0, PB1, PB13, PB14, PB2, PB3, PB4, PC12, PC13, PC15, PC16, PC17, PHY_XIN
- net labels removed: PCLK, XIN
- wire segments 745 -> 794
- no-connect marks 10 -> 15
Other:
- moved on the sheet: C59, C60, J8, R38, R39, R40, R42, TP10, TP7, TP8, TP9, U11

Commit message: Updated schematic
Parts:
- removed R54, R64, R70: 120R, Capacitors_SMD:C_0805, symbol R
- added C19: 100nF, Capacitors_SMD:C_0603, symbol C
- added R15: 10k, Capacitors_SMD:C_0603, symbol R
- added R32, R33, R34: 0R, symbol R
- added R41: 27R, Capacitors_SMD:C_0603, symbol R
- added R58, R68, R75: 150R, Capacitors_SMD:C_0805, symbol R
- R10, R9: value 120R -> 150R
- R12: renamed from R13; value 10k -> 100k
- R14: value 10k -> 100k
- R18: renamed from R17; value 10k -> 100k
- R23: renamed from R22; value 10k -> 100k
- R52: renamed from R48; value 120R -> 150R
- gave numbers to parts that had none: 2
- renumbered C21 to C18, C18 to C20, C19 to C21, C20 to C22, C25 to C23, C22 to C24, C23 to C25, C24 to C26, C26 to C27, C27 to C28, C28 to C29, C29 to C30, C30 to C31, C31 to C32, C32 to C33, C33 to C34, C34 to C35, C35 to C36, C36 to C37, C37 to C38, C38 to C39, C39 to C40, C40 to C41, C41 to C42, C42 to C43, C43 to C44, C44 to C45, C45 to C46, C46 to C47, C47 to C48, C48 to C49, C49 to C50, C50 to C51, C51 to C52, C52 to C53, C53 to C54, C54 to C56, C56 to C57, C57 to C58, C58 to C59, C59 to C60, C60 to C61, J8 to J10, R12 to R13, R15 to R16, R16 to R17, R18 to R19, R19 to R20, R20 to R21, R21 to R22, R23 to R24, R24 to R25, R25 to R26, R26 to R27, R27 to R28, R28 to R29, R29 to R30, R30 to R31, R31 to R35, R32 to R36, R33 to R37, R34 to R38, R35 to R39, R36 to R40, R38 to R42, R40 to R43, R42 to R44, R37 to R45, R41 to R46, R43 to R47, R44 to R48, R45 to R49, R46 to R50, R47 to R51, R49 to R53, R50 to R54, R51 to R55, R52 to R56, R53 to R57, R55 to R59, R56 to R60, R57 to R61, R58 to R62, R59 to R63, R60 to R64, R61 to R65, R62 to R66, R63 to R67, R39 to R69, R65 to R70, R66 to R71, R67 to R72, R68 to R73, R69 to R74, R71 to R76, R72 to R77, R73 to R78, R74 to R79
Connections:
- net labels added: ~RST_R
- wire segments 794 -> 804
Other:
- note removed: "TODO: CHECK THESE CAPACITOR VALUES, THEY SEEM A BIT HIGH."
- moved on the sheet: C1, C10, C11, C12, C13, C14, C15, C16, C17, C18, C2, C20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

Commit message: Cleaned up schematic
Connections:
- wire segments 804 -> 1010
Other:
- moved on the sheet: R34

Commit message: Cleaned up schematic more
Connections:
- wire segments 1010 -> 796
