File: Hardware/Processor_Periph/Processor.sch (KiCad schematic (older format))
At the start: 205 parts, among them J1 UART0, J10 JTAGICE3-SWD, J2 5V, J3 USB_OTG, J4 RJ-45_J0006D01BNL, J5 Micro_SD_Card, J6 I2C, J7 PWM, J8 Spare0, J9 Spare1, Q1 BSS806NE, Q2 BSS806NE, Q3 BSS806NE, Q4 BSS806NE, SW1 ~RST, SW2 PB, SW3 PB, U1 TXS0102, U10 ASE-25.000MHZ-LC-T, U11 CY7C1018, U2 LM3671, U3 S25FL127S, U4 PRTR5V0U2X, U5 MIC5365, U6 DSC61XX, U7 DP83848C, U8 ATSAM4E16E, U9 3.0V, Y1 32.768kHz

Commit message: Modified schematic per 5/21 discussion
- Added 2xGPIO expanders & new connectors for interfacing to x4 stepper
motor drivers
- Added buffer for driving PWM outputs to stepper motors
- Added more spare pins & spare pin connectors
- Removed I2C expansion connector (I2C dedicated to GPIO expanders now)
- Cleaned up component values
- Expanded schematic size
- Reannotated entire schematic
- Regenerated schematic PDF

TODO:

- Generate new BOM with new schematic annotation
- Finalize connector footprints
- Begin layout
Parts:
- removed J6: I2C, symbol CONN_01X03
- removed J7: PWM, symbol CONN_02X06
- added C57, C64, C65, C66, C67: 100nF, Capacitors_SMD:C_0603, symbol C
- added C59: 4.7uF, Capacitors_SMD:C_0805, symbol C
- added J10, J11: CONN_MOTOR, symbol CONN_02X14
- added J9: CONN_SPARE, Pin_Headers:Pin_Header_Angled_2x08_Pitch2.54mm, symbol CONN_02X08
- added JP2, JP3: VCC_SEL, Pin_Headers:Pin_Header_Straight_1x03_Pitch2.54mm, symbol Jumper_NC_Dual
- added R100, R101, R102, R103, R104, R93, R94, R95, R96, R97, R98, R99: 10k, Resistors_SMD:R_0603, symbol R
- added U11: 74HC244, symbol 74HC244
- added U13, U14: TCA6424A, Housings_DFN_QFN:QFN-32-1EP_5x5mm_Pitch0.5mm, symbol TCA6424A
- J1: renamed from J2; footprint (none) -> Pin_Headers:Pin_Header_Angled_1x03_Pitch2.54mm
- J2: renamed from J3; footprint (none) -> FritzLib:USB_Micro-B_10103594-0001LF_holes
- J3: renamed from J1; footprint (none) -> Pin_Headers:Pin_Header_Angled_1x04_Pitch2.54mm
- J4: footprint (none) -> FritzLib:J0006D01BNL
- J5: footprint (none) -> FritzLib:MicroSD-Yamaichi-PJS
- J6: renamed from J8; value Spare0 -> CONN_SPARE; footprint (none) -> Pin_Headers:Pin_Header_Angled_2x08_Pitch2.54mm
- J8: renamed from J9; value Spare1 -> CONN_SPARE; footprint (none) -> Pin_Headers:Pin_Header_Angled_2x08_Pitch2.54mm
- JP1: value 5V_SEL -> VCC_SEL; footprint (none) -> Pin_Headers:Pin_Header_Straight_1x03_Pitch2.54mm
- L1: footprint (none) -> FritzLib:CDRH2D14
- L2: footprint (none) -> FritzLib:Inductor_SMD_3.0mm_x_3.0mm
- Q1, Q2, Q3, Q4: footprint (none) -> TO_SOT_Packages_SMD:SOT-23
- SW1: value ~RST -> PB
- TP1, TP2: footprint Measurement_Points:Test_Point_Keystone_5019_Minature -> FritzLib:Test_Point_Keystone_5019_Minature
- TP10: renamed from TP3; footprint Measurement_Points:Test_Point_Keystone_5019_Minature -> FritzLib:Test_Point_Keystone_5019_Minature
- TP11: renamed from TP4; footprint Measurement_Points:Test_Point_Keystone_5019_Minature -> FritzLib:Test_Point_Keystone_5019_Minature
- TP12: renamed from TP14; footprint Measurement_Points:Test_Point_Keystone_5019_Minature -> FritzLib:Test_Point_Keystone_5019_Minature
- TP13: renamed from TP5; footprint Measurement_Points:Test_Point_Keystone_5019_Minature -> FritzLib:Test_Point_Keystone_5019_Minature
- TP14: renamed from TP6; footprint Measurement_Points:Test_Point_Keystone_5019_Minature -> FritzLib:Test_Point_Keystone_5019_Minature
- TP3: renamed from TP7; footprint Measurement_Points:Test_Point_Keystone_5019_Minature -> FritzLib:Test_Point_Keystone_5019_Minature
- TP4: renamed from TP8; footprint Measurement_Points:Test_Point_Keystone_5019_Minature -> FritzLib:Test_Point_Keystone_5019_Minature
- TP5: renamed from TP9; footprint Measurement_Points:Test_Point_Keystone_5019_Minature -> FritzLib:Test_Point_Keystone_5019_Minature
- TP6: renamed from TP10; footprint Measurement_Points:Test_Point_Keystone_5019_Minature -> FritzLib:Test_Point_Keystone_5019_Minature
- TP7: renamed from TP11; footprint Measurement_Points:Test_Point_Keystone_5019_Minature -> FritzLib:Test_Point_Keystone_5019_Minature
- TP8: renamed from TP13; footprint Measurement_Points:Test_Point_Keystone_5019_Minature -> FritzLib:Test_Point_Keystone_5019_Minature
- TP9: renamed from TP12; footprint Measurement_Points:Test_Point_Keystone_5019_Minature -> FritzLib:Test_Point_Keystone_5019_Minature
- U10, U6: footprint (none) -> Crystals:Crystal_SMD_3225-4pin_3.2x2.5mm
- U12: renamed from U11; footprint (none) -> FritzLib:32-SOJ-300mil
- Y1: footprint (none) -> Crystals:Crystal_SMD_MicroCrystal_CC7V-T1A-2pin_3.2x1.5mm
- renumbered C2 to C1, C8 to C10, C14 to C13, C15 to C14, C19 to C15, C13 to C16, C16 to C17, C17 to C18, C18 to C19, C1 to C2, C30 to C23, C31 to C24, C23 to C25, C35 to C26, C24 to C27, C25 to C28, C26 to C29, C6 to C3, C39 to C30, C27 to C31, C28 to C32, C29 to C33, C42 to C34, C32 to C35, C33 to C36, C34 to C37, C43 to C38, C44 to C39, C3 to C4, C36 to C40, C37 to C41, C38 to C42, C45 to C43, C40 to C44, C41 to C45, C7 to C5, C55 to C54, C54 to C55, C57 to C56, C56 to C58, C10 to C6, C58 to C60, C59 to C61, C60 to C62, C61 to C63, C9 to C7, C4 to C8, C5 to C9, D6 to D1, D1 to D2, D2 to D3, D3 to D4, D4 to D5, D5 to D6, J10 to J7, R49 to R1, R56 to R10, R57 to R11, R4 to R12, R5 to R13, R60 to R14, R61 to R15, R62 to R16, R63 to R17, R8 to R18, R6 to R19, R50 to R2, R65 to R20, R66 to R21, R67 to R22, R68 to R23, R7 to R24, R72 to R25, R73 to R26, R74 to R27, R75 to R28, R77 to R29, R51 to R3, R78 to R30, R79 to R31, R80 to R32, R11 to R33, R9 to R34, R10 to R35, R92 to R36, R13 to R37, R16 to R38, R17 to R39, R52 to R4, R12 to R40, R20 to R41, R21 to R42, R14 to R43, R19 to R44, R24 to R45, R22 to R46, R25 to R47, R15 to R48, R27 to R49, R2 to R5, R18 to R50, R29 to R51, R26 to R52, R34 to R53, R28 to R54, R23 to R55, R35 to R56, R30 to R57, R31 to R58, R32 to R59, R1 to R6, R33 to R60, R81 to R61, R82 to R62, R83 to R63, R84 to R64, R85 to R65, R86 to R66, R87 to R67, R88 to R68, R89 to R69, R3 to R7, R90 to R70, R91 to R71, R36 to R72, R37 to R73, R38 to R74, R39 to R75, R41 to R76, R40 to R77, R42 to R78, R46 to R79, R54 to R8, R47 to R80, R43 to R81, R44 to R82, R45 to R83, R48 to R84, R53 to R85, R70 to R86, R58 to R87, R59 to R88, R64 to R89, R55 to R9, R69 to R90, R71 to R91, R76 to R92, U2 to U1, U1 to U2, U4 to U3, U3 to U4
Connections:
- net labels added: GPIO_01_~INT, GPIO_01_~RST, GPIO_23_~INT, GPIO_23_~RST, M0_DCY, M0_DIR, M0_MM0, M0_MM1, M0_MM2, M0_STP, M0_~EN, M0_~FLT, M0_~HOM, M0_~RST, M0_~SLP, M0_~STP, M1_DCY, M1_DIR, M1_MM0, M1_MM1, M1_MM2, M1_STP, M1_~EN, M1_~FLT, M1_~HOM, M1_~RST, M1_~SLP, M1_~STP, M2_DCY, M2_DIR, M2_MM0, M2_MM1, M2_MM2, M2_STP, M2_~EN, M2_~FLT, M2_~HOM, M2_~RST, M2_~SLP, M2_~STP, M3_DCY, M3_DIR, M3_MM0, M3_MM1, M3_MM2, M3_STP, M3_~EN, M3_~FLT, M3_~HOM, M3_~RST, M3_~SLP, M3_~STP, SPARE0, SPARE1, SPARE2, SPARE3, SPARE4, SPARE5, SPARE6, SPARE7, VCCP_01, VCCP_23
- net labels removed: PA1, PA2, PA5, PA6, PWM
- wire segments 817 -> 1024
Other:
- moved on the sheet: C1, C10, C11, C12, C13, C14, C15, C16, C17, C18, C19, C2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
