File: Hardware/StepperDriverBob/StepperDriverBob.sch (KiCad schematic (older format))
At the start: 0 parts

Commit message: Finished stepper break out board schematic
finished up the stepper break out board schematic for the drv8825. I
used the below link as a guide. I still need to fill in some component
values and what not.
https://www.digikey.com/reference-designs/en/motor-control/821
Parts:
- added C? (x2): 100uF, symbol CP1_Small
- added C? (x3): .1uF, symbol C_Small
- added C?: 0.47uF, symbol C_Small
- added C?: .01uF, symbol C_Small
- added C?: CP1_Small, symbol CP1_Small
- added C?: C_Small, symbol C_Small
- added D?: LED, symbol LED
- added D?: nFAULT, symbol Led_Small
- added D?: nHOME, symbol Led_Small
- added D?: Led_Small, symbol Led_Small
- added P? (x2): CONN_01X02, symbol CONN_01X02
- added P?: CONN_01X09, symbol CONN_01X09
- added R?: R, symbol R
- added R?: 1M, symbol R_Small
- added R? (x2): .2, symbol R_Small
- added R? (x2): 50k, symbol R_Small
- added R? (x4): ?, symbol R_Small
- added R?: R_Small, symbol R_Small
- added U1?: DRV8825, symbol DRV8825
Connections:
- new net: D?.2 (A), R?.2 (x4)
- new net: C?.1, U1?.1 (CP1)
- new net: R?.1, R?.2, U1?.12 (AVREF), U1?.13 (BVREF)
- new net: C?.2, U1?.2 (CP2)
- new net: C?.2, R?.1, U1?.3 (VCP)
- new net: R?.1, U1?.6 (ISENA)
- new net: R?.1, U1?.9 (ISENB)
- new net +3V3: C?.1, C?.1, C?.1, P?.1 (P1), R?.1, R?.1, R?.1, R?.1, R?.1, R?.1, U1?.15 (V3P3OUT)
- new net AOUT1: U1?.5 (AOUT1)
- new net AOUT2: U1?.7 (AOUT2)
- new net BOUT1: U1?.10 (BOUT1)
- new net BOUT2: U1?.8 (BOUT2)
- new net DECAY: P?.3 (P3), U1?.19 (DECAY)
- new net DIR: P?.4 (P4), U1?.20 (DIR)
- new net GND: C?.1, C?.2, C?.2, C?.2, C?.2, C?.2, C?.2, D?.1 (K), D?.1 (K), P?.2 (P2), P?.2 (P2), R?.2, R?.2, R?.2, U1?.14 (GND), U1?.28 (GND), U1?.~ (GND)
- new net MODE0: P?.7 (P7), U1?.24 (MODE0)
- new net MODE1: P?.8 (P8), U1?.25 (MODE1)
- new net MODE2: P?.9 (P9), U1?.26 (MODE2)
- new net STEP: P?.6 (P6), U1?.22 (STEP)
- new net VDD: C?.1, C?.1, C?.1, C?.1, C?.2, P?.1 (P1), R?.1, R?.2, U1?.11 (VMB), U1?.4 (VMA)
- new net nENBL: P?.5 (P5), U1?.21 (nENBL)
- new net nFAULT: D?.1 (K), R?.2, U1?.18 (nFAULT)
- new net nHOME: D?.1 (K), R?.2, U1?.27 (nHOME)
- new net nRESET: P?.1 (P1), U1?.16 (nRESET)
- new net nSLEEP: P?.2 (P2), U1?.17 (nSLEEP)
