File: Hardware/StepperDriverBob/StepperDriverBob.sch (KiCad schematic (older format))
At the start: 28 parts, among them U1? DRV8825

Commit message: Updated stepper bob to better fit with style guide
Parts:
- added P4: CONN_01X04, symbol CONN_01X04
- gave numbers to parts that had none: 28
Connections:
- net labels added: +3V3, ~nFAULT~, ~nHOME~, ~nRESET~
- net labels removed: +3.3V
- wire segments 112 -> 116
- no-connect marks 0 -> 1
Other:
- note added: "TODO: Fill in proper resistor and capacitor values"

Commit message: Added/Completed BOM for StepperDriveBob
Parts:
- removed R10, R8: ?, symbol R_Small
- C1, C4, C5: value .1uF -> 100nF; footprint (none) -> Capacitors_SMD:C_0603
- C2, C3: footprint (none) -> Capacitors_SMD:CP_Elec_5x5.3
- C6: value .01uF -> 10nF; footprint (none) -> Capacitors_SMD:C_0603
- C7: value 0.47uF -> 470nF; footprint (none) -> Capacitors_SMD:C_0603
- C8: value C_Small -> 100nF; footprint (none) -> Capacitors_SMD:C_0603
- C9: value CP1_Small -> 100uF; footprint (none) -> Capacitors_SMD:CP_Elec_5x5.3
- D1: value LED -> MOTOR_PWR; footprint (none) -> LEDs:LED_0603
- D2, D3: footprint (none) -> LEDs:LED_0603
- D4: value Led_Small -> 3V3PWR; footprint (none) -> LEDs:LED_0603
- P1, P2: footprint (none) -> Pin_Headers:Pin_Header_Straight_1x02_Pitch2.54mm
- P3: footprint (none) -> Pin_Headers:Pin_Header_Straight_1x09_Pitch2.54mm
- P4: footprint (none) -> Pin_Headers:Pin_Header_Straight_1x04_Pitch2.54mm
- R1: value R -> 50R; footprint (none) -> Resistors_SMD:R_0603
- R2, R3, R4: footprint (none) -> Resistors_SMD:R_0603
- R5, R6: value .2 -> .2R; footprint (none) -> Resistors_SMD:R_0603
- R7: value ? -> 100R; footprint (none) -> Resistors_SMD:R_0603
- R8: renamed from R9; value ? -> 100R; footprint (none) -> Resistors_SMD:R_0603
- R9: renamed from R11; value R_Small -> 100R; footprint (none) -> Resistors_SMD:R_0603
- U1: renamed from U11; footprint (none) -> Housings_SSOP:HTSSOP-28_4.4x9.7mm_Pitch0.65mm_ThermalPad
Connections:
- wire segments 116 -> 104

Commit message: worked on stepper driver bob schematic and pcb layout
Parts:
- removed C2, C9: 100uF, Capacitors_SMD:CP_Elec_5x5.3, symbol CP1_Small
- removed C4, C8: 100nF, Capacitors_SMD:C_0603, symbol C_Small
- removed D4: 3V3PWR, LEDs:LED_0603, symbol Led_Small
- removed P2: CONN_01X02, Pin_Headers:Pin_Header_Straight_1x02_Pitch2.54mm, symbol CONN_01X02
- removed R9: 100R, Resistors_SMD:R_0603, symbol R_Small
Connections:
- net labels removed: nRESET
- wire segments 104 -> 87
Other:
- note added: "TODO: Fill in proper resistor and capacitor values. Update current draw for 3.3V supply to make sure it doesn't exceede acceptable current draw. 3.3V/100k + the two LED current draws"
- note removed: "TODO: Fill in proper resistor and capacitor values"
Changed lines of the file:
@@
-$EndComp
-$Comp
-L C_Small C4
-U 1 1 58CC8E5E
-P 3950 3200
-F 0 "C4" H 3960 3270 50  0000 L CNN
-F 1 "100nF" H 3960 3120 50  0000 L CNN
-F 2 "Capacitors_SMD:C_0603" H 3950 3200 50  0001 C CNN
-F 3 "" H 3950 3200 50  0000 C CNN
-	1    3950 3200
-	1    0    0    -1
 $EndComp
 $Comp
@@
 $EndComp
 $Comp
-L GND #PWR05
-U 1 1 58CC92BC
-P 3950 3400
-F 0 "#PWR05" H 3950 3150 50  0001 C CNN
-F 1 "GND" H 3950 3250 50  0000 C CNN
-F 2 "" H 3950 3400 50  0000 C CNN
-F 3 "" H 3950 3400 50  0000 C CNN
-	1    3950 3400
-	1    0    0    -1
-$EndComp
-$Comp
-L GND #PWR06
-U 1 1 58CC936C
-P 3450 3700
-F 0 "#PWR06" H 3450 3450 50  0001 C CNN
-F 1 "GND" H 3450 3550 50  0000 C CNN
-F 2 "" H 3450 3700 50  0000 C CNN
-F 3 "" H 3450 3700 50  0000 C CNN
-	1    3450 3700
-	1    0    0    -1
-$EndComp
-$Comp
-L VDD #PWR07
+L VDD #PWR05
 U 1 1 58CC9D6D
 P 3450 4850
-F 0 "#PWR07" H 3450 4700 50  0001 C CNN
+F 0 "#PWR05" H 3450 4700 50  0001 C CNN
 F 1 "VDD" H 3450 5000 50  0000 C CNN
 F 2 "" H 3450 4850 50  0000 C CNN
@@
 F 3 "" H 4400 4300 50  0000 C CNN
 	1    4400 4300
-	1    0    0    -1
-$EndComp
-$Comp
-L CP1_Small C2
-U 1 1 58CCB5F3
-P 3450 3550
-F 0 "C2" H 3460 3620 50  0000 L CNN
-F 1 "100uF" H 3460 3470 50  0000 L CNN
-F 2 "Capacitors_SMD:CP_Elec_5x5.3" H 3450 3550 50  0001 C CNN
-F 3 "" H 3450 3550 50  0000 C CNN
-	1    3450 3550
 	1    0    0    -1
 $EndComp
@@
 	6000 4100 6150 4100
 Wire Wire Line
-	4300 3150 4400 3150
-Wire Wire Line
-	4300 3150 4300 3450
-Wire Wire Line
-	4300 3450 4400 3450
+	4150 3450 4400 3450
 Wire Wire Line
 	4600 3750 4600 4150
@@
 Connection ~ 4300 3050
 Wire Wire Line
-	3450 3300 3450 3450
-Wire Wire Line
 	3700 3050 3700 3650
 Connection ~ 4100 3050
-Connection ~ 3450 3350
 Connection ~ 3700 3350
-Wire Wire Line
-	3950 3300 3950 3400
 Wire Wire Line
 	6450 3950 6450 3900
@@
 Connection ~ 4400 4150
 Wire Wire Line
-	3450 3650 3450 3700
-Wire Wire Line
 	3450 3350 3700 3350
-Wire Wire Line
-	3950 3100 3950 3050
-Connection ~ 3950 3050
-Wire Wire Line
-	3950 3350 4300 3350
-Connection ~ 4300 3350
-Connection ~ 3950 3350
 Wire Wire Line
 	7350 2750 7350 2700
@@
 nHOME
 $Comp
-L CONN_01X02 P2
-U 1 1 58CD414E
-P 10650 2650
-F 0 "P2" H 10650 2800 50  0000 C CNN
-F 1 "CONN_01X02" V 10750 2650 50  0000 C CNN
-F 2 "Pin_Headers:Pin_Header_Straight_1x02_Pitch2.54mm" H 10650 2650 50  0001 C CNN
-F 3 "" H 10650 2650 50  0000 C CNN
-	1    10650 2650
-	1    0    0    -1
-$EndComp
-$Comp
 L CONN_01X09 P3
 U 1 1 58CD4FF3
@@
 $EndComp
 Text GLabel 10400 3300 0    50   Output ~ 0
-nRESET
+~nRESET~
 Text GLabel 10400 3400 0    50   Output ~ 0
 nSLEEP
@@
 	10400 4100 10450 4100
 $Comp
-L CP1_Small C9
-U 1 1 58CDB116
-P 10200 2650
-F 0 "C9" H 10210 2720 50  0000 L CNN
-F 1 "100uF" H 10210 2570 50  0000 L CNN
-F 2 "Capacitors_SMD:CP_Elec_5x5.3" H 10200 2650 50  0001 C CNN
-F 3 "" H 10200 2650 50  0000 C CNN
-	1    10200 2650
-	1    0    0    -1
-$EndComp
-$Comp
-L C_Small C8
-U 1 1 58CDB259
-P 10000 2650
-F 0 "C8" H 10010 2720 50  0000 L CNN
-F 1 "100nF" H 10010 2570 50  0000 L CNN
-F 2 "Capacitors_SMD:C_0603" H 10000 2650 50  0001 C CNN
-F 3 "" H 10000 2650 50  0000 C CNN
-	1    10000 2650
-	1    0    0    -1
-$EndComp
-$Comp
-L R_Small R9
-U 1 1 58CDB522
-P 9750 2500
-F 0 "R9" V 9830 2500 50  0000 C CNN
-F 1 "100R" V 9750 2500 50  0000 C CNN
-F 2 "Resistors_SMD:R_0603" H 9750 2500 50  0001 C CNN
-F 3 "" H 9750 2500 50  0000 C CNN
-	1    9750 2500
-	0    -1   -1   0
-$EndComp
-$Comp
-L Led_Small D4
-U 1 1 58CDB763
-P 9450 2650
-F 0 "D4" V 9530 2610 50  0000 R CNN
-F 1 "3V3PWR" V 9450 2610 50  0000 R CNN
-F 2 "LEDs:LED_0603" V 9450 2650 50  0001 C CNN
-F 3 "" V 9450 2650 50  0000 C CNN
-	1    9450 2650
-	0    -1   -1   0
-$EndComp
-Wire Wire Line
-	10450 2500 10450 2600
-Wire Wire Line
-	9850 2500 10450 2500
-Wire Wire Line
-	10000 2500 10000 2550
-Connection ~ 10000 2500
-Wire Wire Line
-	10200 2500 10200 2550
-Connection ~ 10200 2500
-Wire Wire Line
-	9650 2500 9450 2500
-Wire Wire Line
-	9450 2500 9450 2550
-Wire Wire Line
-	9450 2750 9450 2800
-Wire Wire Line
-	9450 2800 10450 2800
-Wire Wire Line
-	10000 2800 10000 2750
-Wire Wire Line
-	10450 2800 10450 2700
-Connection ~ 10000 2800
-Wire Wire Line
-	10200 2750 10200 2800
-Connection ~ 10200 2800
-$Comp
-L GND #PWR08
-U 1 1 58CDD8C5
-P 9950 2850
-F 0 "#PWR08" H 9950 2600 50  0001 C CNN
-F 1 "GND" H 9950 2700 50  0000 C CNN
-F 2 "" H 9950 2850 50  0000 C CNN
-F 3 "" H 9950 2850 50  0000 C CNN
-	1    9950 2850
-	1    0    0    -1
-$EndComp
-Wire Wire Line
-	9950 2850 9950 2800
-Connection ~ 9950 2800
-Wire Wire Line
-	10350 2450 10350 2500
-Connection ~ 10350 2500
-$Comp
-L +3V3 #PWR09
+L +3V3 #PWR06
 U 1 1 58CE15F3
 P 8100 2700
-F 0 "#PWR09" H 8100 2550 50  0001 C CNN
+F 0 "#PWR06" H 8100 2550 50  0001 C CNN
 F 1 "+3V3" H 8100 2840 50  0000 C CNN
 F 2 "" H 8100 2700 50  0000 C CNN
@@
 $EndComp
 $Comp
-L +3V3 #PWR010
+L +3V3 #PWR07
 U 1 1 58CE178B
 P 7350 2700
-F 0 "#PWR010" H 7350 2550 50  0001 C CNN
+F 0 "#PWR07" H 7350 2550 50  0001 C CNN
 F 1 "+3V3" H 7350 2840 50  0000 C CNN
 F 2 "" H 7350 2700 50  0000 C CNN
@@
 $EndComp
 $Comp
-L +3V3 #PWR011
+L +3V3 #PWR08
 U 1 1 58CE1BDF
 P 6450 3900
-F 0 "#PWR011" H 6450 3750 50  0001 C CNN
+F 0 "#PWR08" H 6450 3750 50  0001 C CNN
 F 1 "+3V3" H 6450 4040 50  0000 C CNN
 F 2 "" H 6450 3900 50  0000 C CNN
@@
 $EndComp
 $Comp
-L +3V3 #PWR012
-U 1 1 58CE10D9
-P 10350 2450
-F 0 "#PWR012" H 10350 2300 50  0001 C CNN
-F 1 "+3V3" H 10350 2590 50  0000 C CNN
-F 2 "" H 10350 2450 50  0000 C CNN
-F 3 "" H 10350 2450 50  0000 C CNN
-	1    10350 2450
-	1    0    0    -1
-$EndComp
-$Comp
-L +3V3 #PWR013
+L +3V3 #PWR09
 U 1 1 58CE287D
 P 4400 3850
-F 0 "#PWR013" H 4400 3700 50  0001 C CNN
+F 0 "#PWR09" H 4400 3700 50  0001 C CNN
 F 1 "+3V3" H 4400 3990 50  0000 C CNN
 F 2 "" H 4400 3850 50  0000 C CNN
@@
 Text GLabel 10400 4650 0    50   Input ~ 0
 AOUT2
+Text GLabel 10400 4750 0    50   Input ~ 0
+BOUT2
 Text GLabel 10400 4850 0    50   Input ~ 0
-BOUT2
-Text GLabel 10400 4750 0    50   Input ~ 0
 BOUT1
 Wire Wire Line
@@
 Wire Wire Line
 	10400 4650 10450 4650
+Text Notes 8000 1800 2    152  ~ 0
+TODO: Fill in proper resistor and capacitor values. Update current draw for 3.3V supply to make sure it doesn't exceede acceptable current draw. 3.3V/100k + the two LED current draws
+Wire Wire Line
+	7350 3200 7350 3250
+Wire Wire Line
+	8100 3200 8100 3250
+Wire Wire Line
+	3450 3300 3450 3350
+$Comp
+L GND #PWR010
+U 1 1 58F27C48
+P 4150 3450
+F 0 "#PWR010" H 4150 3200 50  0001 C CNN
+F 1 "GND" H 4150 3300 50  0000 C CNN
+F 2 "" H 4150 3450 50  0000 C CNN
+F 3 "" H 4150 3450 50  0000 C CNN
+	1    4150 3450
+	1    0    0    -1
+$EndComp
+$Comp
+L GND #PWR011
+U 1 1 58F27C84
+P 4300 3200
+F 0 "#PWR011" H 4300 2950 50  0001 C CNN
+F 1 "GND" H 4300 3050 50  0000 C CNN
+F 2 "" H 4300 3200 50  0000 C CNN
+F 3 "" H 4300 3200 50  0000 C CNN
+	1    4300 3200
+	1    0    0    -1
+$EndComp
+Wire Wire Line
+	4400 3150 4300 3150
+Wire Wire Line
+	4300 3150 4300 3200
 Wire Wire Line
 	10400 4750 10450 4750
 Wire Wire Line
 	10400 4850 10450 4850
-Text Notes 8000 1800 2    152  ~ 0
-TODO: Fill in proper resistor and capacitor values
-Wire Wire Line
-	7350 3200 7350 3250
-Wire Wire Line
-	8100 3200 8100 3250
 $EndSCHEMATC

Commit message: Finished pcb layout
-drv8825.lib connected thermal pad to ground
-changed global labels to local labels for readability
-finsihed routing pcb(just need to do ground plane.
Parts:
- D1: symbol LED -> LED-RESCUE-StepperDriverBob
- D2: value nFAULT -> ~FAULT~
- D3: value nHOME -> ~HOME~
- R3, R4: footprint Resistors_SMD:R_0603 -> Pin_Headers:Pin_Header_Straight_1x02_Pitch2.54mm
- U1: symbol DRV8825 -> DRV8825-RESCUE-StepperDriverBob
Connections:
- net labels added: A0UT2, ~ENBL~, ~FAULT~, ~HOME~, ~RST~, ~SLEEP~
- net labels removed: AOUT2, nENBL, nFAULT, nHOME, nSLEEP, ~nFAULT~, ~nHOME~, ~nRESET~

Commit message: Finished up pcb routing
+Holdes for standoffs
+Made the board larger 1.7x.1.7 in
+Rerouted entire board
Parts:
- added C2: 100nF, Capacitors_SMD:C_0603, symbol C_Small
- R3: renamed from R5; footprint Resistors_SMD:R_0603 -> Resistors_SMD:R_2010
- R4: renamed from R6; footprint Resistors_SMD:R_0603 -> Resistors_SMD:R_2010
- renumbered C3 to C1, C5 to C3, C1 to C4, C6 to C5, C7 to C6, P3 to P2, P4 to P3, R3 to R5, R4 to R6
Connections:
- wire segments 87 -> 89
Other:
- moved on the sheet: C1, C4, R5, R6

Commit message: Added pins for fault and home outpouts
Parts:
- removed P2: CONN_01X09, Pin_Headers:Pin_Header_Straight_1x09_Pitch2.54mm, symbol CONN_01X09
- added J1: CONN_01X11, Pin_Headers:Pin_Header_Straight_1x11_Pitch2.54mm, symbol CONN_01X11
- renumbered P3 to P2
Connections:
- wire segments 89 -> 91
Changed lines of the file:
@@
 $EndDescr
 $Comp
-L GND #PWR10
+L GND #PWR01
 U 1 1 58CB9AF3
 P 5400 4550
-F 0 "#PWR10" H 5400 4300 50  0001 C CNN
+F 0 "#PWR01" H 5400 4300 50  0001 C CNN
 F 1 "GND" H 5400 4400 50  0000 C CNN
 F 2 "" H 5400 4550 50  0000 C CNN
@@
 $EndComp
 $Comp
-L GND #PWR2
+L GND #PWR02
 U 1 1 58CBE0D0
 P 3350 5400
-F 0 "#PWR2" H 3350 5150 50  0001 C CNN
+F 0 "#PWR02" H 3350 5150 50  0001 C CNN
 F 1 "GND" H 3350 5250 50  0000 C CNN
 F 2 "" H 3350 5400 50  0000 C CNN
@@
 $EndComp
 $Comp
-L GND #PWR9
+L GND #PWR03
 U 1 1 58CC6A6B
 P 4550 4750
-F 0 "#PWR9" H 4550 4500 50  0001 C CNN
+F 0 "#PWR03" H 4550 4500 50  0001 C CNN
 F 1 "GND" H 4550 4600 50  0000 C CNN
 F 2 "" H 4550 4750 50  0000 C CNN
@@
 $EndComp
 $Comp
-L VDD #PWR3
+L VDD #PWR04
 U 1 1 58CC9205
 P 3450 3300
-F 0 "#PWR3" H 3450 3150 50  0001 C CNN
+F 0 "#PWR04" H 3450 3150 50  0001 C CNN
 F 1 "VDD" H 3450 3450 50  0000 C CNN
 F 2 "" H 3450 3300 50  0000 C CNN
@@
 $EndComp
 $Comp
-L VDD #PWR1
+L VDD #PWR05
 U 1 1 58CC9D6D
 P 3350 4850
-F 0 "#PWR1" H 3350 4700 50  0001 C CNN
+F 0 "#PWR05" H 3350 4700 50  0001 C CNN
 F 1 "VDD" H 3350 5000 50  0000 C CNN
 F 2 "" H 3350 4850 50  0000 C CNN
@@
 $EndComp
 $Comp
-L CONN_01X09 P2
-U 1 1 58CD4FF3
-P 10650 3700
-F 0 "P2" H 10650 4200 50  0000 C CNN
-F 1 "CONN_01X09" V 10750 3700 50  0000 C CNN
-F 2 "Pin_Headers:Pin_Header_Straight_1x09_Pitch2.54mm" H 10650 3700 50  0001 C CNN
-F 3 "" H 10650 3700 50  0000 C CNN
-	1    10650 3700
-	1    0    0    -1
-$EndComp
-$Comp
-L +3V3 #PWR13
+L +3V3 #PWR06
 U 1 1 58CE15F3
 P 8100 2700
-F 0 "#PWR13" H 8100 2550 50  0001 C CNN
+F 0 "#PWR06" H 8100 2550 50  0001 C CNN
 F 1 "+3V3" H 8100 2840 50  0000 C CNN
 F 2 "" H 8100 2700 50  0000 C CNN
@@
 $EndComp
 $Comp
-L +3V3 #PWR12
+L +3V3 #PWR07
 U 1 1 58CE178B
 P 7350 2700
-F 0 "#PWR12" H 7350 2550 50  0001 C CNN
+F 0 "#PWR07" H 7350 2550 50  0001 C CNN
 F 1 "+3V3" H 7350 2840 50  0000 C CNN
 F 2 "" H 7350 2700 50  0000 C CNN
@@
 $EndComp
 $Comp
-L +3V3 #PWR11
+L +3V3 #PWR08
 U 1 1 58CE1BDF
 P 6450 3900
-F 0 "#PWR11" H 6450 3750 50  0001 C CNN
+F 0 "#PWR08" H 6450 3750 50  0001 C CNN
 F 1 "+3V3" H 6450 4040 50  0000 C CNN
 F 2 "" H 6450 3900 50  0000 C CNN
@@
 $EndComp
 $Comp
-L +3V3 #PWR8
+L +3V3 #PWR09
 U 1 1 58CE287D
 P 4550 4150
-F 0 "#PWR8" H 4550 4000 50  0001 C CNN
+F 0 "#PWR09" H 4550 4000 50  0001 C CNN
 F 1 "+3V3" H 4550 4290 50  0000 C CNN
 F 2 "" H 4550 4150 50  0000 C CNN
@@
 NoConn ~ 5950 3150
 $Comp
-L CONN_01X04 P3
+L CONN_01X04 P2
 U 1 1 58CE360C
 P 10650 4700
-F 0 "P3" H 10650 4950 50  0000 C CNN
+F 0 "P2" H 10650 4950 50  0000 C CNN
 F 1 "CONN_01X04" V 10750 4700 50  0000 C CNN
 F 2 "Pin_Headers:Pin_Header_Straight_1x04_Pitch2.54mm" H 10650 4700 50  0001 C CNN
@@
 TODO: Fill in proper resistor and capacitor values. Update current draw for 3.3V supply to make sure it doesn't exceede acceptable current draw. 3.3V/100k + the two LED current draws
 $Comp
-L GND #PWR5
+L GND #PWR010
 U 1 1 58F27C48
 P 4150 3450
-F 0 "#PWR5" H 4150 3200 50  0001 C CNN
+F 0 "#PWR010" H 4150 3200 50  0001 C CNN
 F 1 "GND" H 4150 3300 50  0000 C CNN
 F 2 "" H 4150 3450 50  0000 C CNN
@@
 $EndComp
 $Comp
-L GND #PWR7
+L GND #PWR011
 U 1 1 58F27C84
 P 4300 3200
-F 0 "#PWR7" H 4300 2950 50  0001 C CNN
+F 0 "#PWR011" H 4300 2950 50  0001 C CNN
 F 1 "GND" H 4300 3050 50  0000 C CNN
 F 2 "" H 4300 3200 50  0000 C CNN
@@
 Text Label 8100 3250 3    60   ~ 0
 ~HOME~
+Text Label 10400 3200 2    60   ~ 0
+~RST~
 Text Label 10400 3300 2    60   ~ 0
-~RST~
-Text Label 10400 3400 2    60   ~ 0
 ~SLEEP~
 Wire Wire Line
@@
 Connection ~ 4250 3650
 $Comp
-L GND #PWR6
+L GND #PWR012
 U 1 1 59067F78
 P 4250 3950
-F 0 "#PWR6" H 4250 3700 50  0001 C CNN
+F 0 "#PWR012" H 4250 3700 50  0001 C CNN
 F 1 "GND" H 4250 3800 50  0000 C CNN
 F 2 "" H 4250 3950 50  0001 C CNN
@@
 Connection ~ 4000 3050
 $Comp
-L GND #PWR4
+L GND #PWR013
 U 1 1 590683DA
 P 4000 3350
-F 0 "#PWR4" H 4000 3100 50  0001 C CNN
+F 0 "#PWR013" H 4000 3100 50  0001 C CNN
 F 1 "GND" H 4000 3200 50  0000 C CNN
 F 2 "" H 4000 3350 50  0001 C CNN
@@
 Wire Wire Line
 	4000 3300 4000 3350
+Wire Wire Line
+	10450 3200 10100 3200
+Wire Wire Line
+	10450 4200 10100 4200
+Text Label 10400 4200 2    60   ~ 0
+~HOME~
+Text Label 10400 3400 2    60   ~ 0
+~FAULT~
+$Comp
+L CONN_01X11 J1
+U 1 1 59069DC8
+P 10650 3700
+F 0 "J1" H 10650 4300 50  0000 C CNN
+F 1 "CONN_01X11" V 10750 3700 50  0000 C CNN
+F 2 "Pin_Headers:Pin_Header_Straight_1x11_Pitch2.54mm" H 10650 3700 50  0001 C CNN
+F 3 "" H 10650 3700 50  0001 C CNN
+	1    10650 3700
+	1    0    0    -1
+$EndComp
 $EndSCHEMATC

Commit message: Finishing Touches
+added holes for offset in schmatic so they wouldn't disspear upon
reloading netlist
+added through holdes to make sure ground planes are connected
+updated silkscreen labels
+moved some components around so that silk screen labels identified them
more easily
Parts:
- added TP1: MOUNT1, Mounting_Holes:MountingHole_3.2mm_M3_Pad, symbol TEST
- added TP2: MOUNT2, Mounting_Holes:MountingHole_3.2mm_M3_Pad, symbol TEST
- added TP3: MOUNT3, Mounting_Holes:MountingHole_3.2mm_M3_Pad, symbol TEST
- added TP4: MOUNT4, Mounting_Holes:MountingHole_3.2mm_M3_Pad, symbol TEST
Changed lines of the file:
@@
 $EndDescr
 $Comp
-L GND #PWR01
+L GND #PWR10
 U 1 1 58CB9AF3
 P 5400 4550
-F 0 "#PWR01" H 5400 4300 50  0001 C CNN
+F 0 "#PWR10" H 5400 4300 50  0001 C CNN
 F 1 "GND" H 5400 4400 50  0000 C CNN
 F 2 "" H 5400 4550 50  0000 C CNN
@@
 $EndComp
 $Comp
-L GND #PWR02
+L GND #PWR2
 U 1 1 58CBE0D0
 P 3350 5400
-F 0 "#PWR02" H 3350 5150 50  0001 C CNN
+F 0 "#PWR2" H 3350 5150 50  0001 C CNN
 F 1 "GND" H 3350 5250 50  0000 C CNN
 F 2 "" H 3350 5400 50  0000 C CNN
@@
 $EndComp
 $Comp
-L GND #PWR03
+L GND #PWR9
 U 1 1 58CC6A6B
 P 4550 4750
-F 0 "#PWR03" H 4550 4500 50  0001 C CNN
+F 0 "#PWR9" H 4550 4500 50  0001 C CNN
 F 1 "GND" H 4550 4600 50  0000 C CNN
 F 2 "" H 4550 4750 50  0000 C CNN
@@
 $EndComp
 $Comp
-L VDD #PWR04
+L VDD #PWR3
 U 1 1 58CC9205
 P 3450 3300
-F 0 "#PWR04" H 3450 3150 50  0001 C CNN
+F 0 "#PWR3" H 3450 3150 50  0001 C CNN
 F 1 "VDD" H 3450 3450 50  0000 C CNN
 F 2 "" H 3450 3300 50  0000 C CNN
@@
 $EndComp
 $Comp
-L VDD #PWR05
+L VDD #PWR1
 U 1 1 58CC9D6D
 P 3350 4850
-F 0 "#PWR05" H 3350 4700 50  0001 C CNN
+F 0 "#PWR1" H 3350 4700 50  0001 C CNN
 F 1 "VDD" H 3350 5000 50  0000 C CNN
 F 2 "" H 3350 4850 50  0000 C CNN
@@
 $EndComp
 $Comp
-L +3V3 #PWR06
+L +3V3 #PWR13
 U 1 1 58CE15F3
 P 8100 2700
-F 0 "#PWR06" H 8100 2550 50  0001 C CNN
+F 0 "#PWR13" H 8100 2550 50  0001 C CNN
 F 1 "+3V3" H 8100 2840 50  0000 C CNN
 F 2 "" H 8100 2700 50  0000 C CNN
@@
 $EndComp
 $Comp
-L +3V3 #PWR07
+L +3V3 #PWR12
 U 1 1 58CE178B
 P 7350 2700
-F 0 "#PWR07" H 7350 2550 50  0001 C CNN
+F 0 "#PWR12" H 7350 2550 50  0001 C CNN
 F 1 "+3V3" H 7350 2840 50  0000 C CNN
 F 2 "" H 7350 2700 50  0000 C CNN
@@
 $EndComp
 $Comp
-L +3V3 #PWR08
+L +3V3 #PWR11
 U 1 1 58CE1BDF
 P 6450 3900
-F 0 "#PWR08" H 6450 3750 50  0001 C CNN
+F 0 "#PWR11" H 6450 3750 50  0001 C CNN
 F 1 "+3V3" H 6450 4040 50  0000 C CNN
 F 2 "" H 6450 3900 50  0000 C CNN
@@
 $EndComp
 $Comp
-L +3V3 #PWR09
+L +3V3 #PWR8
 U 1 1 58CE287D
 P 4550 4150
-F 0 "#PWR09" H 4550 4000 50  0001 C CNN
+F 0 "#PWR8" H 4550 4000 50  0001 C CNN
 F 1 "+3V3" H 4550 4290 50  0000 C CNN
 F 2 "" H 4550 4150 50  0000 C CNN
@@
 TODO: Fill in proper resistor and capacitor values. Update current draw for 3.3V supply to make sure it doesn't exceede acceptable current draw. 3.3V/100k + the two LED current draws
 $Comp
-L GND #PWR010
+L GND #PWR5
 U 1 1 58F27C48
 P 4150 3450
-F 0 "#PWR010" H 4150 3200 50  0001 C CNN
+F 0 "#PWR5" H 4150 3200 50  0001 C CNN
 F 1 "GND" H 4150 3300 50  0000 C CNN
 F 2 "" H 4150 3450 50  0000 C CNN
@@
 $EndComp
 $Comp
-L GND #PWR011
+L GND #PWR7
 U 1 1 58F27C84
 P 4300 3200
-F 0 "#PWR011" H 4300 2950 50  0001 C CNN
+F 0 "#PWR7" H 4300 2950 50  0001 C CNN
 F 1 "GND" H 4300 3050 50  0000 C CNN
 F 2 "" H 4300 3200 50  0000 C CNN
@@
 Connection ~ 4250 3650
 $Comp
-L GND #PWR012
+L GND #PWR6
 U 1 1 59067F78
 P 4250 3950
-F 0 "#PWR012" H 4250 3700 50  0001 C CNN
+F 0 "#PWR6" H 4250 3700 50  0001 C CNN
 F 1 "GND" H 4250 3800 50  0000 C CNN
 F 2 "" H 4250 3950 50  0001 C CNN
@@
 Connection ~ 4000 3050
 $Comp
-L GND #PWR013
+L GND #PWR4
 U 1 1 590683DA
 P 4000 3350
-F 0 "#PWR013" H 4000 3100 50  0001 C CNN
+F 0 "#PWR4" H 4000 3100 50  0001 C CNN
 F 1 "GND" H 4000 3200 50  0000 C CNN
 F 2 "" H 4000 3350 50  0001 C CNN
@@
 	1    0    0    -1
 $EndComp
+$Comp
+L TEST TP1
+U 1 1 5906A0F4
+P 1250 2600
+F 0 "TP1" H 1250 2900 50  0000 C BNN
+F 1 "MOUNT1" H 1250 2850 50  0000 C CNN
+F 2 "Mounting_Holes:MountingHole_3.2mm_M3_Pad" H 1250 2600 50  0001 C CNN
+F 3 "" H 1250 2600 50  0001 C CNN
+	1    1250 2600
+	1    0    0    -1
+$EndComp
+$Comp
+L TEST TP2
+U 1 1 5906A4FB
+P 1600 2600
+F 0 "TP2" H 1600 2900 50  0000 C BNN
+F 1 "MOUNT2" H 1600 2850 50  0000 C CNN
+F 2 "Mounting_Holes:MountingHole_3.2mm_M3_Pad" H 1600 2600 50  0001 C CNN
+F 3 "" H 1600 2600 50  0001 C CNN
+	1    1600 2600
+	1    0    0    -1
+$EndComp
+$Comp
+L TEST TP3
+U 1 1 5906A558
+P 1950 2600
+F 0 "TP3" H 1950 2900 50  0000 C BNN
+F 1 "MOUNT3" H 1950 2850 50  0000 C CNN
+F 2 "Mounting_Holes:MountingHole_3.2mm_M3_Pad" H 1950 2600 50  0001 C CNN
+F 3 "" H 1950 2600 50  0001 C CNN
+	1    1950 2600
+	1    0    0    -1
+$EndComp
+$Comp
+L TEST TP4
+U 1 1 5906A5BE
+P 2300 2600
+F 0 "TP4" H 2300 2900 50  0000 C BNN
+F 1 "MOUNT4" H 2300 2850 50  0000 C CNN
+F 2 "Mounting_Holes:MountingHole_3.2mm_M3_Pad" H 2300 2600 50  0001 C CNN
+F 3 "" H 2300 2600 50  0001 C CNN
+	1    2300 2600
+	1    0    0    -1
+$EndComp
