File: Hardware/StepperDriverBob/StepperDriverBob.sch (KiCad schematic (older format))
At the start: 25 parts, among them J1 CONN_01X11, P1 CONN_01X02, P2 CONN_01X04, U1 DRV8825

Commit message: Ordered Rev1
+added 2 100ohm resistor in place of 50 ohm
Parts:
- added R1: 100R, Resistors_SMD:R_0603, symbol R
- R2: renamed from R1; value 50R -> 100R
- renumbered R2 to R3, R3 to R4, R4 to R5, R5 to R6, R6 to R7, R7 to R8, R8 to R9
Connections:
- wire segments 91 -> 93
- no-connect marks 1 -> 5
Other:
- note removed: "TODO: Fill in proper resistor and capacitor values. Update current draw for 3.3V supply to make sure it doesn't exceede acceptable current draw. 3.3V/100k + the two LED current draws"
- moved on the sheet: R2
Changed lines of the file:
@@
 $EndDescr
 $Comp
-L GND #PWR10
+L GND #PWR01
 U 1 1 58CB9AF3
 P 5400 4550
-F 0 "#PWR10" H 5400 4300 50  0001 C CNN
+F 0 "#PWR01" H 5400 4300 50  0001 C CNN
 F 1 "GND" H 5400 4400 50  0000 C CNN
 F 2 "" H 5400 4550 50  0000 C CNN
@@
 $EndComp
 $Comp
-L R R1
+L R R2
 U 1 1 58CBDE1A
-P 3050 4950
-F 0 "R1" V 3130 4950 50  0000 C CNN
-F 1 "50R" V 3050 4950 50  0000 C CNN
-F 2 "Resistors_SMD:R_0603" V 2980 4950 50  0001 C CNN
-F 3 "" H 3050 4950 50  0000 C CNN
-	1    3050 4950
+P 3050 5050
+F 0 "R2" V 3130 5050 50  0000 C CNN
+F 1 "100R" V 3050 5050 50  0000 C CNN
+F 2 "Resistors_SMD:R_0603" V 2980 5050 50  0001 C CNN
+F 3 "" H 3050 5050 50  0000 C CNN
+	1    3050 5050
 	0    -1   -1   0
 $EndComp
@@
 $EndComp
 $Comp
-L GND #PWR2
+L GND #PWR02
 U 1 1 58CBE0D0
 P 3350 5400
-F 0 "#PWR2" H 3350 5150 50  0001 C CNN
+F 0 "#PWR02" H 3350 5150 50  0001 C CNN
 F 1 "GND" H 3350 5250 50  0000 C CNN
 F 2 "" H 3350 5400 50  0000 C CNN
@@
 $EndComp
 $Comp
-L GND #PWR9
+L GND #PWR03
 U 1 1 58CC6A6B
 P 4550 4750
-F 0 "#PWR9" H 4550 4500 50  0001 C CNN
+F 0 "#PWR03" H 4550 4500 50  0001 C CNN
 F 1 "GND" H 4550 4600 50  0000 C CNN
 F 2 "" H 4550 4750 50  0000 C CNN
@@
 $EndComp
 $Comp
-L R_Small R2
+L R_Small R3
 U 1 1 58CC8085
 P 4300 2900
-F 0 "R2" H 4330 2920 50  0000 L CNN
+F 0 "R3" H 4330 2920 50  0000 L CNN
 F 1 "1M" H 4330 2860 50  0000 L CNN
 F 2 "Resistors_SMD:R_0603" H 4300 2900 50  0001 C CNN
@@
 $EndComp
 $Comp
-L R_Small R3
+L R_Small R4
 U 1 1 58CC8663
 P 4500 3150
-F 0 "R3" V 4580 3150 50  0000 C CNN
+F 0 "R4" V 4580 3150 50  0000 C CNN
 F 1 ".2R" V 4500 3150 50  0000 C CNN
 F 2 "Resistors_SMD:R_2010" H 4500 3150 50  0001 C CNN
@@
 $EndComp
 $Comp
-L R_Small R4
+L R_Small R5
 U 1 1 58CC86B5
 P 4500 3450
-F 0 "R4" V 4580 3450 50  0000 C CNN
+F 0 "R5" V 4580 3450 50  0000 C CNN
 F 1 ".2R" V 4500 3450 50  0000 C CNN
 F 2 "Resistors_SMD:R_2010" H 4500 3450 50  0001 C CNN
@@
 $EndComp
 $Comp
-L VDD #PWR3
+L VDD #PWR04
 U 1 1 58CC9205
 P 3450 3300
-F 0 "#PWR3" H 3450 3150 50  0001 C CNN
+F 0 "#PWR04" H 3450 3150 50  0001 C CNN
 F 1 "VDD" H 3450 3450 50  0000 C CNN
 F 2 "" H 3450 3300 50  0000 C CNN
@@
 $EndComp
 $Comp
-L VDD #PWR1
+L VDD #PWR05
 U 1 1 58CC9D6D
 P 3350 4850
-F 0 "#PWR1" H 3350 4700 50  0001 C CNN
+F 0 "#PWR05" H 3350 4700 50  0001 C CNN
 F 1 "VDD" H 3350 5000 50  0000 C CNN
 F 2 "" H 3350 4850 50  0000 C CNN
@@
 $EndComp
 $Comp
-L R_Small R5
+L R_Small R6
 U 1 1 58CCA910
 P 4550 4300
-F 0 "R5" H 4580 4320 50  0000 L CNN
+F 0 "R6" H 4580 4320 50  0000 L CNN
 F 1 "50k" H 4580 4260 50  0000 L CNN
 F 2 "Pin_Headers:Pin_Header_Straight_1x02_Pitch2.54mm" H 4550 4300 50  0001 C CNN
@@
 $EndComp
 $Comp
-L R_Small R6
+L R_Small R7
 U 1 1 58CCA995
 P 4550 4600
-F 0 "R6" H 4580 4620 50  0000 L CNN
+F 0 "R7" H 4580 4620 50  0000 L CNN
 F 1 "50k" H 4580 4560 50  0000 L CNN
 F 2 "Pin_Headers:Pin_Header_Straight_1x02_Pitch2.54mm" H 4550 4600 50  0001 C CNN
@@
 $EndComp
 $Comp
-L R_Small R7
+L R_Small R8
 U 1 1 58CCCE55
 P 7350 2850
-F 0 "R7" H 7380 2870 50  0000 L CNN
+F 0 "R8" H 7380 2870 50  0000 L CNN
 F 1 "100R" H 7380 2810 50  0000 L CNN
 F 2 "Resistors_SMD:R_0603" H 7350 2850 50  0001 C CNN
@@
 $EndComp
 $Comp
-L R_Small R8
+L R_Small R9
 U 1 1 58CD2500
 P 8100 2850
-F 0 "R8" H 8130 2870 50  0000 L CNN
+F 0 "R9" H 8130 2870 50  0000 L CNN
 F 1 "100R" H 8130 2810 50  0000 L CNN
 F 2 "Resistors_SMD:R_0603" H 8100 2850 50  0001 C CNN
@@
 $EndComp
 $Comp
-L +3V3 #PWR13
+L +3V3 #PWR06
 U 1 1 58CE15F3
 P 8100 2700
-F 0 "#PWR13" H 8100 2550 50  0001 C CNN
+F 0 "#PWR06" H 8100 2550 50  0001 C CNN
 F 1 "+3V3" H 8100 2840 50  0000 C CNN
 F 2 "" H 8100 2700 50  0000 C CNN
@@
 $EndComp
 $Comp
-L +3V3 #PWR12
+L +3V3 #PWR07
 U 1 1 58CE178B
 P 7350 2700
-F 0 "#PWR12" H 7350 2550 50  0001 C CNN
+F 0 "#PWR07" H 7350 2550 50  0001 C CNN
 F 1 "+3V3" H 7350 2840 50  0000 C CNN
 F 2 "" H 7350 2700 50  0000 C CNN
@@
 $EndComp
 $Comp
-L +3V3 #PWR11
+L +3V3 #PWR08
 U 1 1 58CE1BDF
 P 6450 3900
-F 0 "#PWR11" H 6450 3750 50  0001 C CNN
+F 0 "#PWR08" H 6450 3750 50  0001 C CNN
 F 1 "+3V3" H 6450 4040 50  0000 C CNN
 F 2 "" H 6450 3900 50  0000 C CNN
@@
 $EndComp
 $Comp
-L +3V3 #PWR8
+L +3V3 #PWR09
 U 1 1 58CE287D
 P 4550 4150
-F 0 "#PWR8" H 4550 4000 50  0001 C CNN
+F 0 "#PWR09" H 4550 4000 50  0001 C CNN
 F 1 "+3V3" H 4550 4290 50  0000 C CNN
 F 2 "" H 4550 4150 50  0000 C CNN
@@
 	1    0    0    -1
 $EndComp
-Text Notes 8000 1800 2    152  ~ 0
-TODO: Fill in proper resistor and capacitor values. Update current draw for 3.3V supply to make sure it doesn't exceede acceptable current draw. 3.3V/100k + the two LED current draws
-$Comp
-L GND #PWR5
+$Comp
+L GND #PWR010
 U 1 1 58F27C48
 P 4150 3450
-F 0 "#PWR5" H 4150 3200 50  0001 C CNN
+F 0 "#PWR010" H 4150 3200 50  0001 C CNN
 F 1 "GND" H 4150 3300 50  0000 C CNN
 F 2 "" H 4150 3450 50  0000 C CNN
@@
 $EndComp
 $Comp
-L GND #PWR7
+L GND #PWR011
 U 1 1 58F27C84
 P 4300 3200
-F 0 "#PWR7" H 4300 2950 50  0001 C CNN
+F 0 "#PWR011" H 4300 2950 50  0001 C CNN
 F 1 "GND" H 4300 3050 50  0000 C CNN
 F 2 "" H 4300 3200 50  0000 C CNN
@@
 Connection ~ 4250 3650
 $Comp
-L GND #PWR6
+L GND #PWR012
 U 1 1 59067F78
 P 4250 3950
-F 0 "#PWR6" H 4250 3700 50  0001 C CNN
+F 0 "#PWR012" H 4250 3700 50  0001 C CNN
 F 1 "GND" H 4250 3800 50  0000 C CNN
 F 2 "" H 4250 3950 50  0001 C CNN
@@
 Connection ~ 4000 3050
 $Comp
-L GND #PWR4
+L GND #PWR013
 U 1 1 590683DA
 P 4000 3350
-F 0 "#PWR4" H 4000 3100 50  0001 C CNN
+F 0 "#PWR013" H 4000 3100 50  0001 C CNN
 F 1 "GND" H 4000 3200 50  0000 C CNN
 F 2 "" H 4000 3350 50  0001 C CNN
@@
 	1    0    0    -1
 $EndComp
+NoConn ~ 1250 2600
+NoConn ~ 1600 2600
+NoConn ~ 1950 2600
+NoConn ~ 2300 2600
+$Comp
+L R R1
+U 1 1 5906D58F
+P 3050 4850
+F 0 "R1" V 3130 4850 50  0000 C CNN
+F 1 "100R" V 3050 4850 50  0000 C CNN
+F 2 "Resistors_SMD:R_0603" V 2980 4850 50  0001 C CNN
+F 3 "" H 3050 4850 50  0000 C CNN
+	1    3050 4850
+	0    -1   -1   0
+$EndComp
+Wire Wire Line
+	3200 4850 3200 5050
+Connection ~ 3200 4950
+Wire Wire Line
+	2900 4850 2900 5050
+Connection ~ 2900 4950
 $EndSCHEMATC
